File: v1/pm.kicad_sch (KiCad schematic)
At the start: 42 parts, among them J1 USB_C_Receptacle_USB2.0_16P, Q1 FS8205A, U1 DW01A, U2 MCP73871-2CC, U3 TPS63000, U4 USBLC6-2SC6, U5 SI1016X-T1-GE3

Commit message: Updated layout
Parts:
- removed R17: 100k, Resistor_SMD:R_0603_1608Metric_Pad0.98x0.95mm_HandSolder, symbol Device:R
- removed TP4: 3.3v, TestPoint:TestPoint_Pad_2.0x2.0mm, symbol Connector:TestPoint_Probe
- removed TP6: USB_BAT_AUTO, TestPoint:TestPoint_Pad_2.0x2.0mm, symbol Connector:TestPoint_Probe
- added C19, C26: 0.1uf, Capacitor_SMD:C_0402_1005Metric_Pad0.74x0.62mm_HandSolder, symbol Device:C
- added F2: 1.5A 1206L150THWR, Fuse:Fuse_1206_3216Metric, symbol Device:Fuse
- added G1: GND_TP, TestPoint:TestPoint_Pad_D2.5mm, symbol Connector:TestPoint_Probe
- added P1: 3.3V TP, TestPoint:TestPoint_Pad_D2.5mm, symbol Connector:TestPoint_Probe
- BT1: footprint Connector_JST:JST_PH_B2B-PH-SM4-TB_1x02-1MP_P2.00mm_Vertical -> Battery_Library:4.2v_battery_mount
- C9: footprint Capacitor_SMD:C_0603_1608Metric_Pad1.08x0.95mm_HandSolder -> Capacitor_SMD:C_1210_3225Metric_Pad1.33x2.70mm_HandSolder
- F1: value 1A 1206L050YR -> 1.5A 1206L150THWR
- L1: LCSC Part Name (none) -> https://robu.in/product/swpa4030s2r2mt-sunlord-2-2uh-2-95a-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
- R18, R22: value 0.1 -> 0
Connections:
- net 3.3V_PWR: now also P1.1
- net AUTO_SWTCH_5V: now also R22.2; no longer R22.1, R8.1
- net B+: now also F2.1; no longer BT1.1 (+)
- net B-: now also BT1.1 (-); no longer BT1.2 (-)
- net GND: now also C19.2, C26.2, G1.1
- net GPIO_PG: now also C26.1
- net GPIO_STAT1: now also C19.1
- net AUTO_PATH_PWR: now reaches U3.5 (VIN)
- net AUTO_PATH_PWR: now also R22.1, R8.2; no longer R22.2
- net at C5.1, U3.6 (EN), U3.8 (VINA): now also R8.1; no longer R8.2
- net GPIO_STAT2 renamed STAT2
- net USB_5V_PWR renamed USB_5V_FUSE_PROT
- new net: BT1.2 (+), F2.2
- no-connect marks 3 -> 4
Other:
- moved on the sheet: R16, R22, R8
